Commit message: Using sysfs for the hardware

File: ros2_ws/src/robot_description/urdf/base.xacro (robot description, xacro)
@@ -5,8 +5,4 @@
     <xacro:property name="base_height" value="0.15"/>
     <xacro:property name="base_mass" value="4.0"/>
-    <xacro:property name="base_color" value="0.25 0.25 0.25 1"/>
-    <material name="base_material">
-        <color rgba="${base_color}"/>
-    </material>
     <link name="base_footprint"/>
     <link name="base_link">
@@ -16,5 +12,4 @@
                 <box size="0.195 0.145 0.055"/>
             </geometry>
-            <material name="base_material"/>
         </visual>
         <collision>
@@ -62,5 +57,5 @@
         <parent link="base_footprint"/>
         <child link="base_link"/>
-        <origin xyz="0 0 0.12"/>
+        <origin xyz="0 0 0.1825"/>
     </joint>
 </robot>

File: ros2_ws/src/robot_description/urdf/robot_urdf.xacro (robot description, xacro)
@@ -1,8 +1,6 @@
 <?xml version="1.0"?>
 <robot name="WALL-E" xmlns:xacro="http://www.ros.org/wiki/xacro">
-  <xacro:include filename="$(find robot_description)/world/robot/base.xacro"/>
-  <xacro:include filename="$(find robot_description)/world/robot/wheels.xacro"/>
-  <xacro:include filename="$(find robot_description)/world/robot/sensors.xacro"/>
-  <xacro:include filename="$(find robot_description)/world/robot/ros2_control.xacro"/>
-  <xacro:include filename="$(find robot_description)/world/robot/gazebo_references.xacro"/>
+  <xacro:include filename="$(find robot_description)/urdf/base.xacro"/>
+  <xacro:include filename="$(find robot_description)/urdf/wheels.xacro"/>
+  <xacro:include filename="$(find robot_description)/urdf/ros2_control.xacro"/>
 </robot>

File: ros2_ws/src/robot_description/urdf/wheels.xacro (robot description, xacro)
@@ -11,5 +11,5 @@
     <xacro:property name="rear_wheel_mass"       value="0.1"/>
     <!-- Ackermann geometry (must match controllers.yaml) -->
-    <xacro:property name="wheelbase"            value="0.245"/>   <!-- front-to-rear axle distance -->
+    <!-- <xacro:property name="wheelbase"            value="0.245"/>   front-to-rear axle distance -->
     <xacro:property name="front_track_width"    value="0.23"/>   <!-- left-to-right wheel distance -->
     <xacro:property name="rear_track_width"     value="0.08"/>
@@ -24,7 +24,4 @@
     <xacro:property name="steer_mass"    value="0.05"/>
     <xacro:property name="steer_inertia" value="0.0001"/>
-    <material name="wheel_material">
-        <color rgba="0.1 0.1 0.1 1"/>
-    </material>
     <!-- ==================== -->
     <!-- ===== Macros ===== -->
@@ -52,5 +49,4 @@
                 <origin xyz="0 0 0" rpy="1.5707963 0 0"/>
                 <geometry><cylinder radius="${front_wheel_radius}" length="${front_wheel_width}"/></geometry>
-                <material name="wheel_material"/>
             </visual>
             <collision>
@@ -72,5 +68,4 @@
                 <origin xyz="0 0 0" rpy="1.5707963 0 0"/>
                 <geometry><cylinder radius="${rear_wheel_radius}" length="${rear_wheel_width}"/></geometry>
-                <material name="wheel_material"/>
             </visual>
             <collision>
