Commit message: Starting working on the controller manager

File: ros2_ws/src/hardware/ros2_control.xacro (robot description, xacro)
@@ -1,22 +1,40 @@
-<ros2_control name="LeftWheel" type="actuator">
+<ros2_control name="AckermannSystem" type="system">
   <hardware>
     <plugin>motor_driver/MotorDriver</plugin>
     <param name="pwm_device">/dev/pwmchip0</param>
+  </hardware>
+  <joint name="front_left_steering_joint">
+    <command_interface name="position"/>
+    <state_interface name="position"/>
+    <state_interface name="effort"/>
     <param name="pwm_channel">0</param>
-  </hardware>
+  </joint>
+  <joint name="front_right_steering_joint">
+    <command_interface name="position"/>
+    <state_interface name="position"/>
+    <state_interface name="effort"/>
+    <param name="pwm_channel">1</param>
+  </joint>
   <joint name="front_left_wheel_joint">
     <command_interface name="velocity"/>
     <state_interface name="velocity"/>
+    <state_interface name="effort"/>
+    <param name="pwm_channel">2</param>
+  </joint>
+    <joint name="front_right_wheel_joint">
+    <command_interface name="velocity"/>
+    <state_interface name="velocity"/>
+    <state_interface name="effort"/>
+    <param name="pwm_channel">3</param>
+  </joint>
+  <joint name="rear_left_wheel_joint">
+    <state_interface name="position"/>
+    <state_interface name="velocity"/>
+    <state_interface name="effort"/>
+  </joint>
+    <joint name="rear_right_wheel_joint">
+    <state_interface name="position"/>
+    <state_interface name="velocity"/>
+    <state_interface name="effort"/>
   </joint>
 </ros2_control>
-<ros2_control name="RightWheel" type="actuator">
-  <hardware>
-    <plugin>motor_driver/MotorDriver</plugin>
-    <param name="pwm_device">/dev/pwmchip0</param>
-    <param name="pwm_channel">1</param>
-  </hardware>
-  <joint name="front_right_wheel_joint">
-    <command_interface name="velocity"/>
-    <state_interface name="velocity"/>
-  </joint>
-</ros2_control>

Commit message: Ackermann steering controller work

File: ros2_ws/src/hardware/ros2_control.xacro (robot description, xacro)
@@ -1,40 +1,43 @@
-<ros2_control name="AckermannSystem" type="system">
-  <hardware>
-    <plugin>motor_driver/MotorDriver</plugin>
-    <param name="pwm_device">/dev/pwmchip0</param>
-  </hardware>
-  <joint name="front_left_steering_joint">
-    <command_interface name="position"/>
-    <state_interface name="position"/>
-    <state_interface name="effort"/>
-    <param name="pwm_channel">0</param>
-  </joint>
-  <joint name="front_right_steering_joint">
-    <command_interface name="position"/>
-    <state_interface name="position"/>
-    <state_interface name="effort"/>
-    <param name="pwm_channel">1</param>
-  </joint>
-  <joint name="front_left_wheel_joint">
-    <command_interface name="velocity"/>
-    <state_interface name="velocity"/>
-    <state_interface name="effort"/>
-    <param name="pwm_channel">2</param>
-  </joint>
-    <joint name="front_right_wheel_joint">
-    <command_interface name="velocity"/>
-    <state_interface name="velocity"/>
-    <state_interface name="effort"/>
-    <param name="pwm_channel">3</param>
-  </joint>
-  <joint name="rear_left_wheel_joint">
-    <state_interface name="position"/>
-    <state_interface name="velocity"/>
-    <state_interface name="effort"/>
-  </joint>
-    <joint name="rear_right_wheel_joint">
-    <state_interface name="position"/>
-    <state_interface name="velocity"/>
-    <state_interface name="effort"/>
-  </joint>
-</ros2_control>
+<?xml version="1.0"?>
+<robot name="ros2_control" xmlns:xacro="http://www.ros.org/wiki/xacro">
+  <ros2_control name="AckermannSystem" type="system">
+    <hardware>
+      <plugin>motor_driver/MotorDriver</plugin>
+      <param name="pwm_device">/sys/class/pwm/pwmchip0</param>
+    </hardware>
+    <joint name="front_left_steering_joint">
+      <command_interface name="position"/>
+      <state_interface name="position"/>
+      <state_interface name="effort"/>
+      <param name="pwm_channel">0</param>
+    </joint>
+    <joint name="front_right_steering_joint">
+      <command_interface name="position"/>
+      <state_interface name="position"/>
+      <state_interface name="effort"/>
+      <param name="pwm_channel">1</param>
+    </joint>
+    <joint name="front_left_wheel_joint">
+      <command_interface name="velocity"/>
+      <state_interface name="velocity"/>
+      <state_interface name="effort"/>
+      <param name="pwm_channel">2</param>
+    </joint>
+      <joint name="front_right_wheel_joint">
+      <command_interface name="velocity"/>
+      <state_interface name="velocity"/>
+      <state_interface name="effort"/>
+      <param name="pwm_channel">3</param>
+    </joint>
+    <joint name="rear_left_wheel_joint">
+      <state_interface name="position"/>
+      <state_interface name="velocity"/>
+      <state_interface name="effort"/>
+    </joint>
+      <joint name="rear_right_wheel_joint">
+      <state_interface name="position"/>
+      <state_interface name="velocity"/>
+      <state_interface name="effort"/>
+    </joint>
+  </ros2_control>
+</robot>

File: ros2_ws/src/robot_description/urdf/robot_urdf.xacro (robot description, xacro)
@@ -3,4 +3,4 @@
   <xacro:include filename="$(find robot_description)/urdf/base.xacro"/>
   <xacro:include filename="$(find robot_description)/urdf/wheels.xacro"/>
-  <xacro:include filename="$(find robot_description)/urdf/ros2_control.xacro"/>
+  <xacro:include filename="$(find hardware)/ros2_control.xacro"/>
 </robot>

Commit message: Adding the 4 In pins

File: ros2_ws/src/hardware/ros2_control.xacro (robot description, xacro)
@@ -5,4 +5,7 @@
       <plugin>motor_driver/MotorDriver</plugin>
       <param name="pwm_device">/sys/class/pwm/pwmchip0</param>
+      <!-- GPIO sysfs base offset. Find with: cat /sys/class/gpio/gpiochip*/base /sys/class/gpio/gpiochip*/label -->
+      <!-- Pi 5 RP1 chip is typically 571. Set to 0 if sysfs uses raw BCM numbers. -->
+      <param name="gpio_chip_base">0</param>
     </hardware>
     <joint name="front_left_steering_joint">
@@ -10,5 +13,4 @@
       <state_interface name="position"/>
       <state_interface name="effort"/>
-      <param name="pwm_channel">0</param>
     </joint>
     <joint name="front_right_steering_joint">
@@ -16,17 +18,23 @@
       <state_interface name="position"/>
       <state_interface name="effort"/>
-      <param name="pwm_channel">1</param>
     </joint>
+    <!-- Left motor: ENA=PWM ch0 (GPIO12/pin32), IN1=GPIO27 (pin13), IN2=GPIO22 (pin15) -->
     <joint name="front_left_wheel_joint">
       <command_interface name="velocity"/>
       <state_interface name="velocity"/>
       <state_interface name="effort"/>
-      <param name="pwm_channel">2</param>
+      <param name="pwm_channel">0</param>
+      <param name="in1_gpio">27</param>
+      <param name="in2_gpio">22</param>
     </joint>
-      <joint name="front_right_wheel_joint">
+    <!-- Right motor: ENB not connected yet. IN3=GPIO23 (pin16), IN4=??? -->
+    <!-- WARNING: Physical pin 17 is 3.3V POWER, not a GPIO! Verify your wiring! -->
+    <joint name="front_right_wheel_joint">
       <command_interface name="velocity"/>
       <state_interface name="velocity"/>
       <state_interface name="effort"/>
-      <param name="pwm_channel">3</param>
+      <param name="pwm_channel">1</param>
+      <param name="in1_gpio">23</param>
+      <param name="in2_gpio">24</param>
     </joint>
     <joint name="rear_left_wheel_joint">
