Commit message: Add imu

File: AutonomousWarfare/AutonomousWarfare/ros2_ws/src/robot_description/urdf/sensors.xacro (robot description, xacro)
@@ -18,3 +18,9 @@
     <origin xyz="0 0 0.045"/>
   </joint>
+  <link name="imu_link"/>
+  <joint name="imu_joint" type="fixed">
+    <parent link="base_link"/>
+    <child link="imu_link"/>
+    <origin xyz="0 0 0.1" rpy="0 0 0"/>
+  </joint>
 </robot>
