Commit message: nav2 works completely with RVIZ, gazebo and teleop. lets go!!!

File: ETZ_ws/src/robot_description/world/robot/ros2_control.xacro (robot description, xacro)
@@ -1,32 +1,43 @@
 <?xml version="1.0"?>
 <robot name="ros2_control" xmlns:xacro="http://www.ros.org/wiki/xacro">
+  <!-- Ackermann drivetrain: front steering knuckles are position-actuated by
+       ackermann_steering_controller, rear wheels are velocity-actuated.
+       Front wheel joints are state-only - they free-roll under physics. -->
+  <ros2_control name="GazeboSystem" type="system">
+    <hardware>
+      <plugin>gazebo_ros2_control/GazeboSystem</plugin>
+    </hardware>
+    <joint name="front_left_steering_joint">
+      <command_interface name="position"/>
+      <state_interface name="position"/>
+      <state_interface name="velocity"/>
+    </joint>
+    <joint name="front_right_steering_joint">
+      <command_interface name="position"/>
+      <state_interface name="position"/>
+      <state_interface name="velocity"/>
+    </joint>
+    <joint name="rear_left_wheel_joint">
+      <command_interface name="velocity"/>
+      <state_interface name="position"/>
+      <state_interface name="velocity"/>
+    </joint>
+    <joint name="rear_right_wheel_joint">
+      <command_interface name="velocity"/>
+      <state_interface name="position"/>
+      <state_interface name="velocity"/>
+    </joint>
+    <joint name="front_left_wheel_joint">
+      <state_interface name="position"/>
+      <state_interface name="velocity"/>
+    </joint>
+    <joint name="front_right_wheel_joint">
+      <state_interface name="position"/>
+      <state_interface name="velocity"/>
+    </joint>
+  </ros2_control>
   <gazebo>
-    <plugin name="gazebo_ros_diff_drive" filename="libgazebo_ros_diff_drive.so">
-      <ros>
-        <namespace>/</namespace>
-      </ros>
-      <update_rate>100.0</update_rate>
-      <left_joint>rear_left_wheel_joint</left_joint>
-      <right_joint>rear_right_wheel_joint</right_joint>
-      <wheel_separation>0.08</wheel_separation>
-      <wheel_diameter>0.10</wheel_diameter>
-      <command_topic>cmd_vel_nav</command_topic>
-      <odometry_topic>odom</odometry_topic>
-      <robot_base_frame>base_footprint</robot_base_frame>
-      <publish_odom>true</publish_odom>
-      <publish_odom_tf>false</publish_odom_tf>
-      <publish_wheel_tf>true</publish_wheel_tf>
-      <max_wheel_acceleration>5.0</max_wheel_acceleration>
-      <max_wheel_torque>20.0</max_wheel_torque>
-    </plugin>
-    <plugin name="gazebo_ros_joint_state_publisher" filename="libgazebo_ros_joint_state_publisher.so">
-      <ros>
-        <namespace>/</namespace>
-      </ros>
-      <update_rate>30.0</update_rate>
-      <joint_name>front_left_steering_joint</joint_name>
-      <joint_name>front_right_steering_joint</joint_name>
-      <joint_name>front_left_wheel_joint</joint_name>
-      <joint_name>front_right_wheel_joint</joint_name>
+    <plugin name="gazebo_ros2_control" filename="libgazebo_ros2_control.so">
+      <parameters>$(find robot_description)/config/controller_manager.yaml</parameters>
     </plugin>
   </gazebo>
