Commit message: Fix core nav pipeline: IPC host, sim time, contact stiffness, and A* replan cooldown. Robot successfully reaches goal.

File: ETZ_ws/src/robot_description/world/robot/gazebo_references.xacro (robot description, xacro)
@@ -17,6 +17,6 @@
     <mu1>2.0</mu1>
     <mu2>2.0</mu2>
-    <kp>100000.0</kp>
-    <kd>1.0</kd>
+    <kp>500000.0</kp>
+    <kd>10.0</kd>
     <minDepth>0.001</minDepth>
     <maxVel>0.1</maxVel>
@@ -25,6 +25,6 @@
     <mu1>2.0</mu1>
     <mu2>2.0</mu2>
-    <kp>100000.0</kp>
-    <kd>1.0</kd>
+    <kp>500000.0</kp>
+    <kd>10.0</kd>
     <minDepth>0.001</minDepth>
     <maxVel>0.1</maxVel>
@@ -33,6 +33,6 @@
     <mu1>2.0</mu1>
     <mu2>2.0</mu2>
-    <kp>100000.0</kp>
-    <kd>1.0</kd>
+    <kp>500000.0</kp>
+    <kd>10.0</kd>
     <minDepth>0.001</minDepth>
     <maxVel>0.1</maxVel>
@@ -41,6 +41,6 @@
     <mu1>2.0</mu1>
     <mu2>2.0</mu2>
-    <kp>100000.0</kp>
-    <kd>1.0</kd>
+    <kp>500000.0</kp>
+    <kd>10.0</kd>
     <minDepth>0.001</minDepth>
     <maxVel>0.1</maxVel>

File: ETZ_ws/src/robot_description/world/robot/wheels.xacro (robot description, xacro)
@@ -125,4 +125,11 @@
         <axis xyz="0 1 0"/>
         <dynamics damping="0.01" friction="0.0"/>
+        <!-- gazebo_ros2_control's GazeboSystem applies VELOCITY commands via
+             Gazebo's raw Joint::SetVelocity(), which needs an effort/fmax
+             ceiling to actually reach that velocity against any resistance.
+             Without this, the joint motor defaults to near-zero max force,
+             so commanded velocity is accepted but barely any real torque
+             (and thus barely any real motion) is produced. -->
+        <limit effort="5.0" velocity="30.0"/>
     </joint>
     <joint name="front_right_wheel_joint" type="continuous">
@@ -132,4 +139,5 @@
         <axis xyz="0 1 0"/>
         <dynamics damping="0.01" friction="0.0"/>
+        <limit effort="5.0" velocity="30.0"/>
     </joint>
     <!-- Rear wheel joints (continuous: connect directly to base_link, no steering) -->
@@ -140,4 +148,5 @@
         <axis xyz="0 1 0"/>
         <dynamics damping="0.01" friction="0.0"/>
+        <limit effort="5.0" velocity="30.0"/>
     </joint>
     <joint name="rear_right_wheel_joint" type="continuous">
@@ -147,4 +156,5 @@
         <axis xyz="0 1 0"/>
         <dynamics damping="0.01" friction="0.0"/>
+        <limit effort="5.0" velocity="30.0"/>
     </joint>
 </robot>
