Commit message: Integration

File: AutonomousWarfare/AutonomousWarfare/ros2_ws/src/hardware/ros2_control.xacro (robot description, xacro)
@@ -18,4 +18,5 @@
       <state_interface name="effort"/>
       <param name="servo_index">0</param>
+      <param name="trim_rad">-0.47</param>
     </joint>
     <joint name="front_right_steering_joint">
@@ -24,4 +25,5 @@
       <state_interface name="effort"/>
       <param name="servo_index">1</param>
+      <param name="trim_rad">-0.47</param>
     </joint>
     <!-- Left motor: ENA=PWM ch0 (GPIO12/pin32), IN1=GPIO27 (pin13), IN2=GPIO22 (pin15) -->

File: AutonomousWarfare/AutonomousWarfare/ros2_ws/src/robot_description/urdf/wheels.xacro (robot description, xacro)
@@ -102,5 +102,5 @@
         <origin xyz="0.09 ${front_track_width/2} ${front_wheel_z}"/>
         <axis xyz="0 0 1"/>
-        <limit lower="-0.819" upper="0.819" effort="30.0" velocity="30.0"/>
+        <limit lower="-1.1" upper="1.1" effort="30.0" velocity="30.0"/>
         <dynamics damping="0.2" friction="0.0"/>
     </joint>
@@ -110,5 +110,5 @@
         <origin xyz="0.09 ${-front_track_width/2} ${front_wheel_z}"/>
         <axis xyz="0 0 1"/>
-        <limit lower="-0.819" upper="0.819" effort="30.0" velocity="30.0"/>
+        <limit lower="-1.1" upper="1.1" effort="30.0" velocity="30.0"/>
         <dynamics damping="0.2" friction="0.0"/>
     </joint>
